Commit message: Imported upstream version '0.1.0' of 'upstream'

File: share/urdf/pepper.urdf (robot description, URDF)
Before this commit: robot julietteY20MP, 81 links, 80 joints
Links:
- removed link CameraBottom_optical_frame
- removed link CameraDepth_optical_frame
- removed link CameraTop_optical_frame
- link Head: geometry collision mesh filename=package://pepper_meshes/meshes/1.0/HeadPitch_0.10.stl scale=0.1 0.1 0.1; visual mesh filename=package://pepper_meshes/meshes/1.0/HeadPitch.dae scale=0.1 0.1 0.1
- link Hip: geometry collision mesh filename=package://pepper_meshes/meshes/1.0/HipRoll_0.10.stl scale=0.1 0.1 0.1; visual mesh filename=package://pepper_meshes/meshes/1.0/HipRoll.dae scale=0.1 0.1 0.1
- link LBicep: geometry collision mesh filename=package://pepper_meshes/meshes/1.0/LShoulderRoll_0.10.stl scale=0.1 0.1 0.1; visual mesh filename=package://pepper_meshes/meshes/1.0/LShoulderRoll.dae scale=0.1 0.1 0.1
- link LElbow: geometry collision mesh filename=package://pepper_meshes/meshes/1.0/LElbowYaw_0.10.stl scale=0.1 0.1 0.1; visual mesh filename=package://pepper_meshes/meshes/1.0/LElbowYaw.dae scale=0.1 0.1 0.1
- link LFinger11_link: geometry collision mesh filename=package://pepper_meshes/meshes/1.0/LFinger11_0.10.stl scale=0.1 0.1 0.1; visual mesh filename=package://pepper_meshes/meshes/1.0/LFinger11.dae scale=0.1 0.1 0.1
- link LFinger12_link: geometry collision mesh filename=package://pepper_meshes/meshes/1.0/LFinger12_0.10.stl scale=0.1 0.1 0.1; visual mesh filename=package://pepper_meshes/meshes/1.0/LFinger12.dae scale=0.1 0.1 0.1
- link LFinger13_link: geometry collision mesh filename=package://pepper_meshes/meshes/1.0/LFinger13_0.10.stl scale=0.1 0.1 0.1; visual mesh filename=package://pepper_meshes/meshes/1.0/LFinger13.dae scale=0.1 0.1 0.1
- link LFinger21_link: geometry collision mesh filename=package://pepper_meshes/meshes/1.0/LFinger21_0.10.stl scale=0.1 0.1 0.1; visual mesh filename=package://pepper_meshes/meshes/1.0/LFinger21.dae scale=0.1 0.1 0.1
- link LFinger22_link: geometry collision mesh filename=package://pepper_meshes/meshes/1.0/LFinger22_0.10.stl scale=0.1 0.1 0.1; visual mesh filename=package://pepper_meshes/meshes/1.0/LFinger22.dae scale=0.1 0.1 0.1
- link LFinger23_link: geometry collision mesh filename=package://pepper_meshes/meshes/1.0/LFinger23_0.10.stl scale=0.1 0.1 0.1; visual mesh filename=package://pepper_meshes/meshes/1.0/LFinger23.dae scale=0.1 0.1 0.1
- link LFinger31_link: geometry collision mesh filename=package://pepper_meshes/meshes/1.0/LFinger31_0.10.stl scale=0.1 0.1 0.1; visual mesh filename=package://pepper_meshes/meshes/1.0/LFinger31.dae scale=0.1 0.1 0.1
- link LFinger32_link: geometry collision mesh filename=package://pepper_meshes/meshes/1.0/LFinger32_0.10.stl scale=0.1 0.1 0.1; visual mesh filename=package://pepper_meshes/meshes/1.0/LFinger32.dae scale=0.1 0.1 0.1
- link LFinger33_link: geometry collision mesh filename=package://pepper_meshes/meshes/1.0/LFinger33_0.10.stl scale=0.1 0.1 0.1; visual mesh filename=package://pepper_meshes/meshes/1.0/LFinger33.dae scale=0.1 0.1 0.1
- link LFinger41_link: geometry collision mesh filename=package://pepper_meshes/meshes/1.0/LFinger41_0.10.stl scale=0.1 0.1 0.1; visual mesh filename=package://pepper_meshes/meshes/1.0/LFinger41.dae scale=0.1 0.1 0.1
- link LFinger42_link: geometry collision mesh filename=package://pepper_meshes/meshes/1.0/LFinger42_0.10.stl scale=0.1 0.1 0.1; visual mesh filename=package://pepper_meshes/meshes/1.0/LFinger42.dae scale=0.1 0.1 0.1
- link LFinger43_link: geometry collision mesh filename=package://pepper_meshes/meshes/1.0/LFinger43_0.10.stl scale=0.1 0.1 0.1; visual mesh filename=package://pepper_meshes/meshes/1.0/LFinger43.dae scale=0.1 0.1 0.1
- link LForeArm: geometry collision mesh filename=package://pepper_meshes/meshes/1.0/LElbowRoll_0.10.stl scale=0.1 0.1 0.1; visual mesh filename=package://pepper_meshes/meshes/1.0/LElbowRoll.dae scale=0.1 0.1 0.1
- link LShoulder: geometry collision mesh filename=package://pepper_meshes/meshes/1.0/LShoulderPitch_0.10.stl scale=0.1 0.1 0.1; visual mesh filename=package://pepper_meshes/meshes/1.0/LShoulderPitch.dae scale=0.1 0.1 0.1
- link LThumb1_link: geometry collision mesh filename=package://pepper_meshes/meshes/1.0/LThumb1_0.10.stl scale=0.1 0.1 0.1; visual mesh filename=package://pepper_meshes/meshes/1.0/LThumb1.dae scale=0.1 0.1 0.1
- link LThumb2_link: geometry collision mesh filename=package://pepper_meshes/meshes/1.0/LThumb2_0.10.stl scale=0.1 0.1 0.1; visual mesh filename=package://pepper_meshes/meshes/1.0/LThumb2.dae scale=0.1 0.1 0.1
- link Neck: geometry collision mesh filename=package://pepper_meshes/meshes/1.0/HeadYaw_0.10.stl scale=0.1 0.1 0.1; visual mesh filename=package://pepper_meshes/meshes/1.0/HeadYaw.dae scale=0.1 0.1 0.1
- link Pelvis: geometry collision mesh filename=package://pepper_meshes/meshes/1.0/HipPitch_0.10.stl scale=0.1 0.1 0.1; visual mesh filename=package://pepper_meshes/meshes/1.0/HipPitch.dae scale=0.1 0.1 0.1
- link RBicep: geometry collision mesh filename=package://pepper_meshes/meshes/1.0/RShoulderRoll_0.10.stl scale=0.1 0.1 0.1; visual mesh filename=package://pepper_meshes/meshes/1.0/RShoulderRoll.dae scale=0.1 0.1 0.1
- link RElbow: geometry collision mesh filename=package://pepper_meshes/meshes/1.0/RElbowYaw_0.10.stl scale=0.1 0.1 0.1; visual mesh filename=package://pepper_meshes/meshes/1.0/RElbowYaw.dae scale=0.1 0.1 0.1
- link RFinger11_link: geometry collision mesh filename=package://pepper_meshes/meshes/1.0/RFinger11_0.10.stl scale=0.1 0.1 0.1; visual mesh filename=package://pepper_meshes/meshes/1.0/RFinger11.dae scale=0.1 0.1 0.1
- link RFinger12_link: geometry collision mesh filename=package://pepper_meshes/meshes/1.0/RFinger12_0.10.stl scale=0.1 0.1 0.1; visual mesh filename=package://pepper_meshes/meshes/1.0/RFinger12.dae scale=0.1 0.1 0.1
- link RFinger13_link: geometry collision mesh filename=package://pepper_meshes/meshes/1.0/RFinger13_0.10.stl scale=0.1 0.1 0.1; visual mesh filename=package://pepper_meshes/meshes/1.0/RFinger13.dae scale=0.1 0.1 0.1
- link RFinger21_link: geometry collision mesh filename=package://pepper_meshes/meshes/1.0/RFinger21_0.10.stl scale=0.1 0.1 0.1; visual mesh filename=package://pepper_meshes/meshes/1.0/RFinger21.dae scale=0.1 0.1 0.1
- link RFinger22_link: geometry collision mesh filename=package://pepper_meshes/meshes/1.0/RFinger22_0.10.stl scale=0.1 0.1 0.1; visual mesh filename=package://pepper_meshes/meshes/1.0/RFinger22.dae scale=0.1 0.1 0.1
- link RFinger23_link: geometry collision mesh filename=package://pepper_meshes/meshes/1.0/RFinger23_0.10.stl scale=0.1 0.1 0.1; visual mesh filename=package://pepper_meshes/meshes/1.0/RFinger23.dae scale=0.1 0.1 0.1
- link RFinger31_link: geometry collision mesh filename=package://pepper_meshes/meshes/1.0/RFinger31_0.10.stl scale=0.1 0.1 0.1; visual mesh filename=package://pepper_meshes/meshes/1.0/RFinger31.dae scale=0.1 0.1 0.1
- link RFinger32_link: geometry collision mesh filename=package://pepper_meshes/meshes/1.0/RFinger32_0.10.stl scale=0.1 0.1 0.1; visual mesh filename=package://pepper_meshes/meshes/1.0/RFinger32.dae scale=0.1 0.1 0.1
- link RFinger33_link: geometry collision mesh filename=package://pepper_meshes/meshes/1.0/RFinger33_0.10.stl scale=0.1 0.1 0.1; visual mesh filename=package://pepper_meshes/meshes/1.0/RFinger33.dae scale=0.1 0.1 0.1
- link RFinger41_link: geometry collision mesh filename=package://pepper_meshes/meshes/1.0/RFinger41_0.10.stl scale=0.1 0.1 0.1; visual mesh filename=package://pepper_meshes/meshes/1.0/RFinger41.dae scale=0.1 0.1 0.1
- link RFinger42_link: geometry collision mesh filename=package://pepper_meshes/meshes/1.0/RFinger42_0.10.stl scale=0.1 0.1 0.1; visual mesh filename=package://pepper_meshes/meshes/1.0/RFinger42.dae scale=0.1 0.1 0.1
- link RFinger43_link: geometry collision mesh filename=package://pepper_meshes/meshes/1.0/RFinger43_0.10.stl scale=0.1 0.1 0.1; visual mesh filename=package://pepper_meshes/meshes/1.0/RFinger43.dae scale=0.1 0.1 0.1
- link RForeArm: geometry collision mesh filename=package://pepper_meshes/meshes/1.0/RElbowRoll_0.10.stl scale=0.1 0.1 0.1; visual mesh filename=package://pepper_meshes/meshes/1.0/RElbowRoll.dae scale=0.1 0.1 0.1
- link RShoulder: geometry collision mesh filename=package://pepper_meshes/meshes/1.0/RShoulderPitch_0.10.stl scale=0.1 0.1 0.1; visual mesh filename=package://pepper_meshes/meshes/1.0/RShoulderPitch.dae scale=0.1 0.1 0.1
- link RThumb1_link: geometry collision mesh filename=package://pepper_meshes/meshes/1.0/RThumb1_0.10.stl scale=0.1 0.1 0.1; visual mesh filename=package://pepper_meshes/meshes/1.0/RThumb1.dae scale=0.1 0.1 0.1
- link RThumb2_link: geometry collision mesh filename=package://pepper_meshes/meshes/1.0/RThumb2_0.10.stl scale=0.1 0.1 0.1; visual mesh filename=package://pepper_meshes/meshes/1.0/RThumb2.dae scale=0.1 0.1 0.1
- link Tibia: geometry collision mesh filename=package://pepper_meshes/meshes/1.0/KneePitch_0.10.stl scale=0.1 0.1 0.1; visual mesh filename=package://pepper_meshes/meshes/1.0/KneePitch.dae scale=0.1 0.1 0.1
- link WheelB_link: geometry collision mesh filename=package://pepper_meshes/meshes/1.0/WheelB_0.10.stl scale=0.1 0.1 0.1; visual mesh filename=package://pepper_meshes/meshes/1.0/WheelB.dae scale=0.1 0.1 0.1
- link WheelFL_link: geometry collision mesh filename=package://pepper_meshes/meshes/1.0/WheelFL_0.10.stl scale=0.1 0.1 0.1; visual mesh filename=package://pepper_meshes/meshes/1.0/WheelFL.dae scale=0.1 0.1 0.1
- link WheelFR_link: geometry collision mesh filename=package://pepper_meshes/meshes/1.0/WheelFR_0.10.stl scale=0.1 0.1 0.1; visual mesh filename=package://pepper_meshes/meshes/1.0/WheelFR.dae scale=0.1 0.1 0.1
- link l_wrist: geometry collision mesh filename=package://pepper_meshes/meshes/1.0/LWristYaw_0.10.stl scale=0.1 0.1 0.1; visual mesh filename=package://pepper_meshes/meshes/1.0/LWristYaw.dae scale=0.1 0.1 0.1
- link r_wrist: geometry collision mesh filename=package://pepper_meshes/meshes/1.0/RWristYaw_0.10.stl scale=0.1 0.1 0.1; visual mesh filename=package://pepper_meshes/meshes/1.0/RWristYaw.dae scale=0.1 0.1 0.1
- link torso: geometry collision mesh filename=package://pepper_meshes/meshes/1.0/Torso_0.10.stl scale=0.1 0.1 0.1; visual mesh filename=package://pepper_meshes/meshes/1.0/Torso.dae scale=0.1 0.1 0.1
Joints:
- removed joint CameraBottom_optical_frame_joint
- removed joint CameraDepth_optical_frame_joint
- removed joint CameraTop_optical_frame_joint
- joint Head/Touch/Front_sensor_fixedjoint: origin xyz=0.028175 0 0.21267 rpy=0 0.20944 0 -> xyz=0.0275 0 0.1245 rpy=0 -1.1861 0
- joint Head/Touch/Middle_sensor_fixedjoint: origin xyz=0.0041 0 0.2159 rpy=0 -0.0349066 0 -> xyz=-0.004 0 0.125 rpy=3.14159 -1.57079 -3.14159
- joint Head/Touch/Rear_sensor_fixedjoint: origin xyz=-0.03376 0 0.21052 rpy=0 -0.314159 0 -> xyz=-0.033 0 0.1245 rpy=3.14159 -1.33319 -3.14159
- joint LaserSensor/Front_sensor_fixedjoint: origin xyz=0.0562 0 -0.334 rpy=0 0 0 -> xyz=0.0562 0 -0.0692 rpy=0 0.349044 0
- joint LaserSensor/Left_sensor_fixedjoint: origin xyz=-0.018 0.0899 -0.334 rpy=0 0 1.75728367321 -> xyz=-0.018 0.0899 -0.0759 rpy=8.34035e-09 0.191982 1.5708
- joint LaserSensor/Right_sensor_fixedjoint: origin xyz=-0.018 -0.0899 -0.334 rpy=0 0 -1.75728367321 -> xyz=0.018 -0.0899 -0.0759 rpy=4.08851e-07 0.191857 -1.60746

Commit message: Imported upstream version '0.1.1' of 'upstream'

File: share/urdf/pepper.urdf (robot description, URDF)
Before this commit: robot julietteY20MP, 78 links, 77 joints
Links:
- added link CameraBottom_optical_frame
- added link CameraDepth_optical_frame
- added link CameraTop_optical_frame
- added link SurroundingFrontLaser_device_frame
- added link SurroundingLeftLaser_device_frame
- added link SurroundingRightLaser_device_frame
- link LFinger11_link: mass None -> 2e-06
- link LFinger12_link: mass None -> 2e-06
- link LFinger13_link: mass None -> 2e-06
- link LFinger21_link: mass None -> 2e-06
- link LFinger22_link: mass None -> 2e-06
- link LFinger23_link: mass None -> 2e-06
- link LFinger31_link: mass None -> 2e-06
- link LFinger32_link: mass None -> 2e-06
- link LFinger33_link: mass None -> 2e-06
- link LFinger41_link: mass None -> 2e-06
- link LFinger42_link: mass None -> 2e-06
- link LFinger43_link: mass None -> 2e-06
- link LThumb1_link: mass None -> 2e-06
- link LThumb2_link: mass None -> 2e-06
- link RFinger11_link: mass None -> 2e-06
- link RFinger12_link: mass None -> 2e-06
- link RFinger13_link: mass None -> 2e-06
- link RFinger21_link: mass None -> 2e-06
- link RFinger22_link: mass None -> 2e-06
- link RFinger23_link: mass None -> 2e-06
- link RFinger31_link: mass None -> 2e-06
- link RFinger32_link: mass None -> 2e-06
- link RFinger33_link: mass None -> 2e-06
- link RFinger41_link: mass None -> 2e-06
- link RFinger42_link: mass None -> 2e-06
- link RFinger43_link: mass None -> 2e-06
- link RThumb1_link: mass None -> 2e-06
- link RThumb2_link: mass None -> 2e-06
- link l_gripper: mass None -> 2e-06
- link r_gripper: mass None -> 2e-06
Joints:
- added joint CameraBottom_optical_frame_fixedjoint: type fixed, parent CameraBottom_frame, child CameraBottom_optical_frame, origin xyz=0 0 0 rpy=-1.57079632679 0 -1.57079632679
- added joint CameraDepth_optical_frame_fixedjoint: type fixed, parent CameraDepth_frame, child CameraDepth_optical_frame, origin xyz=0 0 0 rpy=-1.57079632679 0 -1.57079632679
- added joint CameraTop_optical_frame_fixedjoint: type fixed, parent CameraTop_frame, child CameraTop_optical_frame, origin xyz=0 0 0 rpy=-1.57079632679 0 -1.57079632679
- added joint LaserSensor/Front_projected_sensor_fixedjoint: type fixed, parent Tibia, child SurroundingFrontLaser_frame, origin xyz=0.0562 0 -0.334 rpy=0 0 0, axis 0 0 0
- added joint LaserSensor/Left_projected_sensor_fixedjoint: type fixed, parent Tibia, child SurroundingLeftLaser_frame, origin xyz=-0.018 0.0899 -0.334 rpy=0 0 1.75728, axis 0 0 0
- added joint LaserSensor/Right_projected_sensor_fixedjoint: type fixed, parent Tibia, child SurroundingRightLaser_frame, origin xyz=-0.018 -0.0899 -0.334 rpy=0 0 -1.75728, axis 0 0 0
- joint Head/Touch/Front_sensor_fixedjoint: origin xyz=0.0275 0 0.1245 rpy=0 -1.1861 0 -> xyz=0.028175 0 0.21267 rpy=0 0.20944 0
- joint Head/Touch/Middle_sensor_fixedjoint: origin xyz=-0.004 0 0.125 rpy=3.14159 -1.57079 -3.14159 -> xyz=0.0041 0 0.2159 rpy=0 -0.0349066 0
- joint Head/Touch/Rear_sensor_fixedjoint: origin xyz=-0.033 0 0.1245 rpy=3.14159 -1.33319 -3.14159 -> xyz=-0.03376 0 0.21052 rpy=0 -0.314159 0
- joint LaserSensor/Front_sensor_fixedjoint: child SurroundingFrontLaser_frame -> SurroundingFrontLaser_device_frame
- joint LaserSensor/Left_sensor_fixedjoint: child SurroundingLeftLaser_frame -> SurroundingLeftLaser_device_frame
- joint LaserSensor/Right_sensor_fixedjoint: child SurroundingRightLaser_frame -> SurroundingRightLaser_device_frame; origin xyz=0.018 -0.0899 -0.0759 rpy=4.08851e-07 0.191857 -1.60746 -> xyz=-0.018 -0.0899 -0.0759 rpy=4.08851e-07 0.191857 -1.60746
